File: hardware/TileGlobeMC_Node/Core.kicad_sch (KiCad schematic)
At the start: 0 parts

Commit message: PCB progress
Parts:
- added BT1: LIR2450, symbol Device:Battery_Cell
- added C1, C12, C2, C3, C9: 4.7u, Capacitor_SMD:C_0402_1005Metric, symbol Device:C_Small
- added C10, C11, C13, C14, C15, C16, C17, C18, C19, C20, C21, C22, C25, C26: 100n, Capacitor_SMD:C_0402_1005Metric, symbol Device:C_Small
- added C23, C24: 15p, Capacitor_SMD:C_0402_1005Metric, symbol Device:C_Small
- added C4, C5, C6, C7: 4.7u, Capacitor_SMD:C_0603_1608Metric, symbol Device:C_Small
- added C8: 22u, Capacitor_SMD:C_0603_1608Metric, symbol Device:C_Small
- added D1, D2, D4: 1N4148WS, Diode_SMD:D_SOD-323_HandSoldering, symbol Diode:1N4148WS
- added D5: 3V, Diode_SMD:D_SOD-323_HandSoldering, symbol Device:D_Zener_Small
- added J1, J3, J5, J7: P_Female, symbol Connector_Generic:Conn_01x05
- added J11: USB_C, Connector_USB:USB_C_Receptacle_GCT_USB4105-xx-A_16P_TopMnt_Horizontal, symbol Connector:USB_C_Receptacle_USB2.0_16P
- added J12, J14, J16, J18: P_Female_Fallback, Connector_PinSocket_2.54mm:PinSocket_1x05_P2.54mm_Horizontal, symbol Connector_Generic:Conn_01x05
- added J13, J15, J17, J19: P_Male_Fallback, Connector_PinHeader_2.54mm:PinHeader_1x05_P2.54mm_Horizontal, symbol Connector_Generic:Conn_01x05
- added J2, J4, J6, J8: P_Male, Project:BC-15-5P380, symbol Connector_Generic_MountingPin:Conn_01x05_MountingPin
- added J9: SWD, Connector_JST:JST_SH_BM03B-SRSS-TB_1x03-1MP_P1.00mm_Vertical, symbol Connector_Generic_MountingPin:Conn_01x03_MountingPin
- added JP1: RESET, TestPoint:TestPoint_2Pads_Pitch2.54mm_Drill0.8mm, symbol Jumper:Jumper_2_Small_Open
- added JP2: USB_BOOT, TestPoint:TestPoint_2Pads_Pitch2.54mm_Drill0.8mm, symbol Jumper:Jumper_2_Small_Open
- added L1: 3.3u, RP2350:L_pol_2016, symbol Project:L_Polarized_Ferrite_Small
- added L2: 1u, Inductor_SMD:L_Wuerth_MAPI-2010, symbol Device:L_Ferrite_Small
- added Q1: 2N7002, Package_TO_SOT_SMD:SOT-23, symbol Transistor_FET:2N7002
- added R1, R10, R4, R7: 300, Capacitor_SMD:C_0603_1608Metric, symbol Device:R_Small
- added R11, R12, R2, R3, R5, R6, R8, R9: 270, Capacitor_SMD:C_0603_1608Metric, symbol Device:R_Small
- added R13, R24: 33, Capacitor_SMD:C_0603_1608Metric, symbol Device:R_Small
- added R14, R15, R36, R37: 10k, Capacitor_SMD:C_0603_1608Metric, symbol Device:R_Small
- added R16: 1.8k, Capacitor_SMD:C_0603_1608Metric, symbol Device:R_Small
- added R17, R18, R19, R22, R23, R28, R29, R34: 100k, Capacitor_SMD:C_0603_1608Metric, symbol Device:R_Small
- added R20: 86.6k, Capacitor_SMD:C_0603_1608Metric, symbol Device:R_Small
- added R21: 390k, Capacitor_SMD:C_0603_1608Metric, symbol Device:R_Small
- added R25, R30: 1k, Capacitor_SMD:C_0603_1608Metric, symbol Device:R_Small
- added R26, R27: 27, Capacitor_SMD:C_0603_1608Metric, symbol Device:R_Small
- added R32, R33: 5.1k, Capacitor_SMD:C_0603_1608Metric, symbol Device:R_Small
- added U1: RP2350_80QFN, RP2350:RP2350-QFN-80-1EP_10x10_P0.4mm_EP3.4x3.4mm_ThermalVias, symbol RP2350:RP2350_80QFN
- added U2: TPS62A01DRL, Package_TO_SOT_SMD:SOT-563, symbol Regulator_Switching:TPS62A01DRL
- added U3: BQ24232RGT, Package_DFN_QFN:VQFN-16-1EP_3x3mm_P0.5mm_EP1.68x1.68mm_ThermalVias, symbol Project:BQ24232RGT
- added U4: ESP-PSRAM64H, Package_SO:SOIC-8_3.9x4.9mm_P1.27mm, symbol Project:ESP-PSRAM64
- added U5: PY25Q128HA-WXH, Package_SON:WSON-8-1EP_6x5mm_P1.27mm_EP3.4x4.3mm, symbol Memory_Flash:W25Q128JVP
- added U6: PY25Q128HA-SSH, Package_SO:SOIC-8_5.3x5.3mm_P1.27mm, symbol Memory_Flash:W25Q128JVS
- added U7: 74AHC1G04, Package_TO_SOT_SMD:SOT-23-5, symbol 74xGxx:74AHC1G04
- added Y1: 12M, Crystal:Crystal_SMD_3225-4Pin_3.2x2.5mm, symbol Device:Crystal_GND24
Connections:
- new net: C23.2, U1.30 (XIN), Y1.1
- new net: C24.2, R25.1, Y1.3
- new net: D1.1 (K), D2.1 (K), D4.1 (K), R34.2, U2.4 (EN)
- new net: J13.3 (Pin_3), J2.3 (Pin_3), R3.1
- new net: J1.4 (Pin_4), J12.4 (Pin_4), R2.1
- new net: C12.1, R24.1, U1.59 (ADC_AVDD)
- new net: J16.4 (Pin_4), J3.4 (Pin_4), R5.1
- new net: JP2.2 (B), R30.1
- new net: D5.1 (K), R23.2, U1.48 (GPIO39)
- new net: R16.1, U3.15 (ITERM)
- new net: J11.A5 (CC1), R33.2
- new net: J11.B5 (CC2), R32.2
- new net: R20.2, R21.1, U2.5 (FB)
- new net: R22.2, U3.7 (PGOOD), U7.2
- new net: R14.2, U3.1 (TS)
- new net: R25.2, U1.31 (XOUT)
- new net: JP1.2 (B), U1.35 (RUN)
- new net: R27.1, U1.66 (USB_DM)
- new net: R26.1, U1.67 (USB_DP)
- new net: J19.3 (Pin_3), J8.3 (Pin_3), R12.1
- new net: J15.3 (Pin_3), J6.3 (Pin_3), R9.1
- new net: J17.3 (Pin_3), J4.3 (Pin_3), R6.1
- new net: Q1.3 (D), R17.1
- new net: L2.1, U2.2 (SW)
- new net: J18.4 (Pin_4), J7.4 (Pin_4), R11.1
- new net: J14.4 (Pin_4), J5.4 (Pin_4), R8.1
- new net +3V3: C13.1, C14.1, C15.1, C16.1, C17.1, C18.1, C19.1, C20.1, C21.1, C22.1, C25.1, C26.1, C3.1, C8.1, L2.2, R13.1, R21.2, R24.2, R28.2, R29.2, R36.2, R37.2, U1.15 (IOVDD), U1.24 (IOVDD), U1.29 (IOVDD), U1.41 (IOVDD), U1.5 (IOVDD), U1.50 (IOVDD), U1.60 (IOVDD), U1.64 (VREG_VIN), U1.68 (USB_OTP_VDD), U1.69 (QSPI_IOVDD), U1.76 (IOVDD), U4.8 (VCC), U5.8 (VCC), U6.8 (VCC)
- new net +BATT: BT1.1 (+), C4.1, R18.2, U3.2 (BAT), U3.3 (BAT)
- new net 3V3_EN_LATCH: D4.2 (A), U1.53 (GPIO42_ADC2)
- new net BAT_ICHG_SAMPLE: R15.2, U1.49 (GPIO40_ADC0), U3.16 (ISET)
- new net BAT_SAMPLE: R17.2, R18.1, U1.52 (GPIO41_ADC1)
- new net BAT_SAMPLE_EN: Q1.1 (G), R19.2, U1.47 (GPIO38)
- new net BAT_~{CHG}: U1.46 (GPIO37), U3.9 (CHG)
- new net BTN_CENTER: U1.42 (GPIO33)
- new net BTN_CENTER_VBUS: D1.2 (A)
- new net GND_CORE: BT1.2 (-), C1.2, C10.2, C11.2, C12.2, C13.2, C14.2, C15.2, C16.2, C17.2, C18.2, C19.2, C2.2, C20.2, C21.2, C22.2, C23.1, C24.1, C25.2, C26.2, C3.2, C4.2, C5.2, C6.1, C7.2, C8.2, C9.2, D5.2 (A), J1.1 (Pin_1), J11.A1 (GND), J11.A12 (GND), J11.B1 (GND), J11.B12 (GND), J11.S1 (SHIELD), J12.1 (Pin_1), J13.1 (Pin_1), J14.1 (Pin_1), J15.1 (Pin_1), J16.1 (Pin_1), J17.1 (Pin_1), J18.1 (Pin_1), J19.1 (Pin_1), J2.5 (Pin_5), J2.MP (MountPin), J3.1 (Pin_1), J4.5 (Pin_5), J4.MP (MountPin), J5.1 (Pin_1), J6.5 (Pin_5), J6.MP (MountPin), J7.1 (Pin_1), J8.5 (Pin_5), J8.MP (MountPin), J9.2 (Pin_2), J9.MP (MountPin), JP1.1 (A), JP2.1 (A), Q1.2 (S), R14.1, R15.1, R16.2, R19.1, R20.1, R32.1, R33.1, R34.1, U1.62 (VREG_PGND), U1.81 (GND), U2.1 (GND), U3.17 (VSS), U3.4 (CE), U3.5 (EN2), U3.8 (VSS), U4.4 (VSS), U5.4 (GND), U5.9 (EP), U6.4 (GND), U7.3 (GND), Y1.2, Y1.4
- new net GPIO0: U1.54 (GPIO43_ADC3)
- new net GPIO1: U1.55 (GPIO44_ADC4)
- new net GPIO2: U1.56 (GPIO45_ADC5)
- new net GPIO3: U1.57 (GPIO46_ADC6)
- new net GPIO4: U1.58 (GPIO47_ADC7)
- new net I2C_SCL: R37.1, U1.45 (GPIO36)
- new net I2C_SDA: R36.1, U1.44 (GPIO35)
- new net LCD_CS: U1.38 (GPIO30)
- new net LCD_DC: U1.37 (GPIO29)
- new net LCD_MOSI: U1.40 (GPIO32)
- new net LCD_SCK: U1.39 (GPIO31)
- new net PA.CA: R1.2, U1.79 (GPIO2)
- new net PA.CAR: J1.2 (Pin_2), J12.2 (Pin_2), R1.1, U1.78 (GPIO1)
- new net PA.CB: J13.2 (Pin_2), J2.4 (Pin_4), U1.4 (GPIO7)
- new net PA.D0: J1.3 (Pin_3), J12.3 (Pin_3), U1.80 (GPIO3)
- new net PA.D1: R2.2, U1.1 (GPIO4)
- new net PA.D2: J13.4 (Pin_4), J2.2 (Pin_2), U1.2 (GPIO5)
- new net PA.D3: R3.2, U1.3 (GPIO6)
- new net PB.CA: R4.2, U1.7 (GPIO9)
- new net PB.CAR: J16.2 (Pin_2), J3.2 (Pin_2), R4.1, U1.6 (GPIO8)
- new net PB.CB: J17.2 (Pin_2), J4.4 (Pin_4), U1.13 (GPIO14)
- new net PB.D0: J16.3 (Pin_3), J3.3 (Pin_3), U1.8 (GPIO10)
- new net PB.D1: R5.2, U1.9 (GPIO11)
- new net PB.D2: J17.4 (Pin_4), J4.2 (Pin_2), U1.11 (GPIO12)
- new net PB.D3: R6.2, U1.12 (GPIO13)
- new net PC.CA: R7.2, U1.16 (GPIO16)
- new net PC.CAR: J14.2 (Pin_2), J5.2 (Pin_2), R7.1, U1.14 (GPIO15)
- new net PC.CB: J15.2 (Pin_2), J6.4 (Pin_4), U1.21 (GPIO21)
- new net PC.D0: J14.3 (Pin_3), J5.3 (Pin_3), U1.17 (GPIO17)
- new net PC.D1: R8.2, U1.18 (GPIO18)
- new net PC.D2: J15.4 (Pin_4), J6.2 (Pin_2), U1.19 (GPIO19)
- new net PC.D3: R9.2, U1.20 (GPIO20)
- new net PD.CA: R10.2, U1.23 (GPIO23)
- new net PD.CAR: J18.2 (Pin_2), J7.2 (Pin_2), R10.1, U1.22 (GPIO22)
- new net PD.CB: J19.2 (Pin_2), J8.4 (Pin_4), U1.36 (GPIO28)
- new net PD.D0: J18.3 (Pin_3), J7.3 (Pin_3), U1.25 (GPIO24)
- new net PD.D1: R11.2, U1.26 (GPIO25)
- new net PD.D2: J19.4 (Pin_4), J8.2 (Pin_2), U1.27 (GPIO26)
- new net PD.D3: R12.2, U1.28 (GPIO27)
- new net PERI_INT: U1.43 (GPIO34)
- new net QMI_CS0: R28.1, R30.2, U1.75 (QSPI_SS), U5.1 (~{CS}), U6.1 (~{CS})
- new net QMI_CS1: R29.1, U1.77 (GPIO0), U4.1 (~{CE})
- new net QMI_SCK: U1.71 (QSPI_SCLK), U4.6 (SCLK), U5.6 (CLK), U6.6 (CLK)
- new net QMI_SD0: U1.72 (QSPI_SD0), U4.5 (SI/SIO), U5.5 (DI/IO_{0}), U6.5 (DI/IO_{0})
- new net QMI_SD1: U1.74 (QSPI_SD1), U4.2 (SO/SIO), U5.2 (DO/IO_{1}), U6.2 (DO/IO_{1})
- new net QMI_SD2: U1.73 (QSPI_SD2), U4.3 (SIO2), U5.3 (~{WP}/IO_{2}), U6.3 (~{WP}/IO_{2})
- new net QMI_SD3: U1.70 (QSPI_SD3), U4.7 (SIO3), U5.7 (~{HOLD}/~{RESET}/IO_{3}), U6.7 (~{HOLD}/~{RESET}/IO_{3})
- new net RP_DVDD: C1.1, C10.1, C11.1, C9.1, L1.1, U1.10 (DVDD), U1.32 (DVDD), U1.51 (DVDD), U1.65 (VREG_FB)
- new net RP_VREG_AVDD: C2.1, R13.2, U1.61 (VREG_AVDD)
- new net RP_VREG_LX: L1.2, U1.63 (VREG_LX)
- new net SWCLK: J9.1 (Pin_1), U1.33 (SWCLK)
- new net SWD: J9.3 (Pin_3), U1.34 (SWD)
- new net USB_D+: J11.A6 (D+), J11.B6 (D+), R26.2
- new net USB_D-: J11.A7 (D-), J11.B7 (D-), R27.2
- new net VBUS: C5.1, C7.1, R22.1, U2.3 (VIN), U3.10 (OUT), U3.11 (OUT), U3.6 (EN1), U7.5 (VCC)
- new net VIN: C6.2, J1.5 (Pin_5), J11.A4 (VBUS), J11.A9 (VBUS), J11.B4 (VBUS), J11.B9 (VBUS), J12.5 (Pin_5), J13.5 (Pin_5), J14.5 (Pin_5), J15.5 (Pin_5), J16.5 (Pin_5), J17.5 (Pin_5), J18.5 (Pin_5), J19.5 (Pin_5), J2.1 (Pin_1), J3.5 (Pin_5), J4.1 (Pin_1), J5.5 (Pin_5), J6.1 (Pin_1), J7.5 (Pin_5), J8.1 (Pin_1), U3.13 (IN)
- new net VIN_PGOOD: D2.2 (A), R23.1, U7.4
- no-connect marks 0 -> 5
Other:
- note added: "3.3V DC-DC"
- note added: "Battery Charger & Power Path"
- note added: "Flash & PSRAM"
- note added: "Node Ports"
- note added: "USB-C"

Commit message: PCB progress
Parts:
- removed D1, D2, D4: 1N4148WS, Diode_SMD:D_SOD-323_HandSoldering, symbol Diode:1N4148WS
- removed J11: USB_C, Connector_USB:USB_C_Receptacle_GCT_USB4105-xx-A_16P_TopMnt_Horizontal, symbol Connector:USB_C_Receptacle_USB2.0_16P
- removed R32, R33: 5.1k, Capacitor_SMD:C_0603_1608Metric, symbol Device:R_Small
- removed R36, R37: 10k, Capacitor_SMD:C_0603_1608Metric, symbol Device:R_Small
- removed U2: TPS62A01DRL, Package_TO_SOT_SMD:SOT-563, symbol Regulator_Switching:TPS62A01DRL
- removed U5: PY25Q128HA-WXH, Package_SON:WSON-8-1EP_6x5mm_P1.27mm_EP3.4x4.3mm, symbol Memory_Flash:W25Q128JVP
- added C36: 120p, Capacitor_SMD:C_0402_1005Metric, symbol Device:C_Small
- added D1, D2, D4: 1N4148WT, Diode_SMD:D_SOD-523, symbol Diode:1N4148WT
- added D10, D11, D12, D13, D14, D15, D16, D17, D18, D19, D20, D21, D22, D23, D24, D25, D26, D27, D28, D29, D6, D7, D8, D9: ESD5Z3.3C, Diode_SMD:D_SOD-523, symbol Diode:ESD5Zxx
- added H1, H2, H3, H4: MountingHole, MountingHole:MountingHole_2.2mm_M2, symbol Mechanical:MountingHole
- added U2: TPS62A01PDDC, Package_TO_SOT_SMD:SOT-23-6, symbol Regulator_Switching:TPS62A01PDDC
- BT1: footprint (none) -> Project:BS-24-B___014; Link (none) -> https://www.lcsc.com/product-detail/C48687361.html
- D5: footprint Diode_SMD:D_SOD-323_HandSoldering -> Diode_SMD:D_SOD-523
- J1, J3, J5, J7: footprint (none) -> Project:BC-20-5PD160
- J12, J14, J16, J18: footprint Connector_PinSocket_2.54mm:PinSocket_1x05_P2.54mm_Horizontal -> Project:PinSocket_1x05_P2.54mm_Horizontal_NoSilk
- J13, J15, J17, J19: footprint Connector_PinHeader_2.54mm:PinHeader_1x05_P2.54mm_Horizontal -> Project:PinHeader_1x05_P2.54mm_Horizontal_NoSilk
- JP1, JP2: footprint TestPoint:TestPoint_2Pads_Pitch2.54mm_Drill0.8mm -> Connector_PinHeader_1.00mm:PinHeader_1x02_P1.00mm_Vertical
- R1, R10, R11, R12, R14, R15, R16, R17, R18, R19, R2, R22, R23, R26, R27, R28, R29, R3, R30, R34, R4, R5, R6, R7, R8, R9: footprint Capacitor_SMD:C_0603_1608Metric -> Resistor_SMD:R_0603_1608Metric
- R13, R20, R21, R24, R25: footprint Capacitor_SMD:C_0603_1608Metric -> Resistor_SMD:R_0402_1005Metric
- U6: now fitted
Connections:
- net BTN_CENTER is gone; now on net GPIO0: U1.42 (GPIO33)
- net I2C_SCL is gone; now on net GPIO3: U1.45 (GPIO36)
- net I2C_SDA is gone; now on net GPIO2: U1.44 (GPIO35)
- net LCD_CS is gone; now on net BAT_~{CHG}: U1.38 (GPIO30)
- net LCD_DC is gone; now on net 3V3_EN_LATCH: U1.37 (GPIO29)
- net LCD_MOSI is gone; now on an unnamed net: U1.40 (GPIO32)
- net LCD_SCK is gone; now on net BAT_SAMPLE_EN: U1.39 (GPIO31)
- net PERI_INT is gone; now on net GPIO1: U1.43 (GPIO34)
- net +3V3: now also C36.1
- net 3V3_EN_LATCH: now also D4.2 (A); no longer U1.53 (GPIO42_ADC2)
- net BAT_ICHG_SAMPLE: now also U1.57 (GPIO46_ADC6); no longer U1.49 (GPIO40_ADC0)
- net BAT_SAMPLE: now also U1.58 (GPIO47_ADC7); no longer U1.52 (GPIO41_ADC1)
- net BAT_SAMPLE_EN: no longer U1.47 (GPIO38)
- net BAT_~{CHG}: no longer U1.46 (GPIO37)
- net BTN_CENTER_VBUS: now also D1.2 (A)
- net GND_CORE: now also J1.5 (Pin_5), J12.5 (Pin_5), J13.5 (Pin_5), J14.5 (Pin_5), J15.5 (Pin_5), J16.5 (Pin_5), J17.5 (Pin_5), J18.5 (Pin_5), J19.5 (Pin_5), J2.1 (Pin_1), J3.5 (Pin_5), J4.1 (Pin_1), J5.5 (Pin_5), J6.1 (Pin_1), J7.5 (Pin_5), J8.1 (Pin_1), D10.2 (A), D11.2 (A), D12.2 (A), D13.2 (A), D14.2 (A), D15.2 (A), D16.2 (A), D17.2 (A), D18.2 (A), D19.2 (A), D20.2 (A), D21.2 (A), D22.2 (A), D23.2 (A), D24.2 (A), D25.2 (A), D26.2 (A), D27.2 (A), D28.2 (A), D29.2 (A), D6.2 (A), D7.2 (A), D8.2 (A), D9.2 (A), U2.2 (GND); no longer J1.1 (Pin_1), J12.1 (Pin_1), J13.1 (Pin_1), J14.1 (Pin_1), J15.1 (Pin_1), J16.1 (Pin_1), J17.1 (Pin_1), J18.1 (Pin_1), J19.1 (Pin_1), J2.5 (Pin_5), J3.1 (Pin_1), J4.5 (Pin_5), J5.1 (Pin_1), J6.5 (Pin_5), J7.1 (Pin_1), J8.5 (Pin_5)
- net GPIO0: no longer U1.54 (GPIO43_ADC3)
- net GPIO1: no longer U1.55 (GPIO44_ADC4)
- net GPIO2: no longer U1.56 (GPIO45_ADC5)
- net GPIO3: no longer U1.57 (GPIO46_ADC6)
- net GPIO4: now also U1.46 (GPIO37); no longer U1.58 (GPIO47_ADC7)
- net PA.CA: now also U1.7 (GPIO9); no longer U1.79 (GPIO2)
- net PA.CAR: now also J13.4 (Pin_4), J2.2 (Pin_2), U1.6 (GPIO8), D6.1 (K); no longer J1.2 (Pin_2), J12.2 (Pin_2), U1.78 (GPIO1)
- net PA.CB: now also J1.4 (Pin_4), J12.4 (Pin_4), U1.13 (GPIO14), D11.1 (K); no longer J13.2 (Pin_2), J2.4 (Pin_4), U1.4 (GPIO7)
- net PA.D0: now also J13.3 (Pin_3), J2.3 (Pin_3), U1.8 (GPIO10), D7.1 (K); no longer J1.3 (Pin_3), J12.3 (Pin_3), U1.80 (GPIO3)
- net PA.D1: now also U1.9 (GPIO11); no longer U1.1 (GPIO4)
- net PA.D2: now also J1.2 (Pin_2), J12.2 (Pin_2), U1.11 (GPIO12), D9.1 (K); no longer J13.4 (Pin_4), J2.2 (Pin_2), U1.2 (GPIO5)
- net PA.D3: now also U1.12 (GPIO13); no longer U1.3 (GPIO6)
- net PB.CA: now also U1.16 (GPIO16); no longer U1.7 (GPIO9)
- net PB.CAR: now also J17.4 (Pin_4), J4.2 (Pin_2), U1.14 (GPIO15), D18.1 (K); no longer J16.2 (Pin_2), J3.2 (Pin_2), U1.6 (GPIO8)
- net PB.CB: now also J16.4 (Pin_4), J3.4 (Pin_4), U1.21 (GPIO21), D23.1 (K); no longer J17.2 (Pin_2), J4.4 (Pin_4), U1.13 (GPIO14)
- net PB.D0: now also J17.3 (Pin_3), J4.3 (Pin_3), U1.17 (GPIO17), D19.1 (K); no longer J16.3 (Pin_3), J3.3 (Pin_3), U1.8 (GPIO10)
- net PB.D1: now also U1.18 (GPIO18); no longer U1.9 (GPIO11)
- net PB.D2: now also J16.2 (Pin_2), J3.2 (Pin_2), U1.19 (GPIO19), D21.1 (K); no longer J17.4 (Pin_4), J4.2 (Pin_2), U1.11 (GPIO12)
- net PB.D3: now also U1.20 (GPIO20); no longer U1.12 (GPIO13)
- net PC.CA: now also U1.23 (GPIO23); no longer U1.16 (GPIO16)
- net PC.CAR: now also J15.4 (Pin_4), J6.2 (Pin_2), U1.22 (GPIO22), D12.1 (K); no longer J14.2 (Pin_2), J5.2 (Pin_2), U1.14 (GPIO15)
- net PC.CB: now also J14.4 (Pin_4), J5.4 (Pin_4), U1.36 (GPIO28), D17.1 (K); no longer J15.2 (Pin_2), J6.4 (Pin_4), U1.21 (GPIO21)
- net PC.D0: now also J15.3 (Pin_3), J6.3 (Pin_3), U1.25 (GPIO24), D13.1 (K); no longer J14.3 (Pin_3), J5.3 (Pin_3), U1.17 (GPIO17)
- net PC.D1: now also U1.26 (GPIO25); no longer U1.18 (GPIO18)
- net PC.D2: now also J14.2 (Pin_2), J5.2 (Pin_2), U1.27 (GPIO26), D15.1 (K); no longer J15.4 (Pin_4), J6.2 (Pin_2), U1.19 (GPIO19)
- net PC.D3: now also U1.28 (GPIO27); no longer U1.20 (GPIO20)
- net PD.CA: now also U1.79 (GPIO2); no longer U1.23 (GPIO23)
- net PD.CAR: now also J19.4 (Pin_4), J8.2 (Pin_2), U1.78 (GPIO1), D24.1 (K); no longer J18.2 (Pin_2), J7.2 (Pin_2), U1.22 (GPIO22)
- net PD.CB: now also J18.4 (Pin_4), J7.4 (Pin_4), U1.4 (GPIO7), D29.1 (K); no longer J19.2 (Pin_2), J8.4 (Pin_4), U1.36 (GPIO28)
- net PD.D0: now also J19.3 (Pin_3), J8.3 (Pin_3), U1.80 (GPIO3), D25.1 (K); no longer J18.3 (Pin_3), J7.3 (Pin_3), U1.25 (GPIO24)
- net PD.D1: now also U1.1 (GPIO4); no longer U1.26 (GPIO25)
- net PD.D2: now also J18.2 (Pin_2), J7.2 (Pin_2), U1.2 (GPIO5), D27.1 (K); no longer J19.4 (Pin_4), J8.2 (Pin_2), U1.27 (GPIO26)
- net PD.D3: now also U1.3 (GPIO6); no longer U1.28 (GPIO27)
- net VBUS: now also U2.4 (VIN)
- net VIN: now also J1.1 (Pin_1), J12.1 (Pin_1), J13.1 (Pin_1), J14.1 (Pin_1), J15.1 (Pin_1), J16.1 (Pin_1), J17.1 (Pin_1), J18.1 (Pin_1), J19.1 (Pin_1), J2.5 (Pin_5), J3.1 (Pin_1), J4.5 (Pin_5), J5.1 (Pin_1), J6.5 (Pin_5), J7.1 (Pin_1), J8.5 (Pin_5); no longer J1.5 (Pin_5), J12.5 (Pin_5), J13.5 (Pin_5), J14.5 (Pin_5), J15.5 (Pin_5), J16.5 (Pin_5), J17.5 (Pin_5), J18.5 (Pin_5), J19.5 (Pin_5), J2.1 (Pin_1), J3.5 (Pin_5), J4.1 (Pin_1), J5.5 (Pin_5), J6.1 (Pin_1), J7.5 (Pin_5), J8.1 (Pin_1)
- net VIN_PGOOD: now also D2.2 (A)
- net at R34.2: now also D1.1 (K), D2.1 (K), D4.1 (K), U2.1 (EN)
- net at D5.1 (K), R23.2: no longer U1.48 (GPIO39)
- net at R20.2, R21.1: now also C36.2, U2.6 (FB)
- net at L2.1: now also U2.3 (SW)
- new net: D8.1 (K), J13.2 (Pin_2), J2.4 (Pin_4), R2.1
- new net: D10.1 (K), J1.3 (Pin_3), J12.3 (Pin_3), R3.1
- new net: D22.1 (K), J16.3 (Pin_3), J3.3 (Pin_3), R6.1
- new net: D20.1 (K), J17.2 (Pin_2), J4.4 (Pin_4), R5.1
- new net: D26.1 (K), J19.2 (Pin_2), J8.4 (Pin_4), R11.1
- new net: D14.1 (K), J15.2 (Pin_2), J6.4 (Pin_4), R8.1
- new net: D28.1 (K), J18.3 (Pin_3), J7.3 (Pin_3), R12.1
- new net: D16.1 (K), J14.3 (Pin_3), J5.3 (Pin_3), R9.1
- new net GPIO10: U1.54 (GPIO43_ADC3)
- new net GPIO11: U1.55 (GPIO44_ADC4)
- new net GPIO12: U1.56 (GPIO45_ADC5)
- new net GPIO5: U1.47 (GPIO38)
- new net GPIO6: U1.48 (GPIO39)
- new net GPIO7: U1.49 (GPIO40_ADC0)
- new net GPIO8: U1.52 (GPIO41_ADC1)
- new net GPIO9: U1.53 (GPIO42_ADC2)
- no-connect marks 5 -> 3
Other:
- note removed: "USB-C"
- moved on the sheet: C8, D5, J1, J12, J13, J14, J15, J16, J17, J18, J19, J2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

Commit message: Main PCB progress
Parts:
- removed JP1: RESET, Connector_PinHeader_1.00mm:PinHeader_1x02_P1.00mm_Vertical, symbol Jumper:Jumper_2_Small_Open
- added TP1: RP_RUN, TestPoint:TestPoint_THTPad_D1.0mm_Drill0.5mm, symbol Connector:TestPoint
- Q1: value 2N7002 -> 2N7002W; footprint Package_TO_SOT_SMD:SOT-23 -> Package_TO_SOT_SMD:SOT-323_SC-70
- R17, R18, R19, R22, R23, R26, R27: footprint Resistor_SMD:R_0603_1608Metric -> Resistor_SMD:R_0402_1005Metric
- U1: footprint RP2350:RP2350-QFN-80-1EP_10x10_P0.4mm_EP3.4x3.4mm_ThermalVias -> Project:RP2350-QFN-80-1EP_10x10_P0.4mm_EP3.4x3.4mm_ThermalVias
- U3: footprint Package_DFN_QFN:VQFN-16-1EP_3x3mm_P0.5mm_EP1.68x1.68mm_ThermalVias -> Project:VQFN-16-1EP_3x3mm_P0.5mm_EP1.68x1.68mm_ThermalVias
- U7: footprint Package_TO_SOT_SMD:SOT-23-5 -> Package_TO_SOT_SMD:SOT-353_SC-70-5
Connections:
- net 3V3_EN_LATCH: now also U1.23 (GPIO23); no longer U1.37 (GPIO29)
- net BAT_SAMPLE_EN: now also U1.40 (GPIO32); no longer U1.39 (GPIO31)
- net BAT_~{CHG}: now also U1.14 (GPIO15); no longer U1.38 (GPIO30)
- net GND_CORE: no longer J9.MP (MountPin)
- net PB.CA: now also U1.17 (GPIO17); no longer U1.16 (GPIO16)
- net PB.CAR: now also U1.16 (GPIO16); no longer U1.14 (GPIO15)
- net PB.CB: now also U1.22 (GPIO22); no longer U1.21 (GPIO21)
- net PB.D0: now also U1.18 (GPIO18); no longer U1.17 (GPIO17)
- net PB.D1: now also U1.19 (GPIO19); no longer U1.18 (GPIO18)
- net PB.D2: now also U1.20 (GPIO20); no longer U1.19 (GPIO19)
- net PB.D3: now also U1.21 (GPIO21); no longer U1.20 (GPIO20)
- net PC.CA: now also U1.26 (GPIO25); no longer U1.23 (GPIO23)
- net PC.CAR: now also U1.25 (GPIO24); no longer U1.22 (GPIO22)
- net PC.CB: now also U1.38 (GPIO30); no longer U1.36 (GPIO28)
- net PC.D0: now also U1.27 (GPIO26); no longer U1.25 (GPIO24)
- net PC.D1: now also U1.28 (GPIO27); no longer U1.26 (GPIO25)
- net PC.D2: now also U1.36 (GPIO28); no longer U1.27 (GPIO26)
- net PC.D3: now also U1.37 (GPIO29); no longer U1.28 (GPIO27)
- net VIN: now also J9.MP (MountPin)
- net at D5.1 (K), R23.2: now also U1.39 (GPIO31); no longer U1.40 (GPIO32)
- net at U1.35 (RUN): now also TP1.1
Other:
- moved on the sheet: D5

Commit message: BOM; PCB minor tweaks
Parts:
- added C37: 100n, Capacitor_SMD:C_0603_1608Metric, symbol Device:C_Small
- C1, C12, C2, C3, C9: Link (none) -> https://www.lcsc.com/product-detail/C368809.html
- C10, C11, C13, C14, C15, C16, C17, C18, C19, C20, C21, C22, C25, C26: Link (none) -> https://www.lcsc.com/product-detail/C60474.html
- C23, C24: Link (none) -> https://www.lcsc.com/product-detail/C326803.html
- C36: Link (none) -> https://www.lcsc.com/product-detail/C45359895.html
- C4, C5, C6, C7: Link (none) -> https://www.lcsc.com/product-detail/C1705.html
- C8: Link (none) -> https://www.lcsc.com/product-detail/C86295.html
- D1, D2, D4: Link (none) -> https://www.lcsc.com/product-detail/C917006.html
- D10, D11, D12, D13, D14, D15, D16, D17, D18, D19, D20, D21, D22, D23, D24, D25, D26, D27, D28, D29, D6, D7, D8, D9: value ESD5Z3.3C -> ESD5Z3.3-HXY; Link (none) -> https://www.lcsc.com/product-detail/C4748782.html
- D5: Link (none) -> https://www.lcsc.com/product-detail/C6771811.html
- H1, H2, H3, H4: now in the parts list
- J1, J3, J5, J7: Link (none) -> https://www.aliexpress.com/item/4000203259512.html
- J12, J14, J16, J18: Link (none) -> https://www.lcsc.com/product-detail/C35167.html
- J13, J15, J17, J19: Link (none) -> https://www.lcsc.com/product-detail/C492413.html
- J2, J4, J6, J8: Link (none) -> https://www.aliexpress.com/item/1005004198626809.html
- J9: Link (none) -> https://www.lcsc.com/product-detail/C7433423.html
- L1: Link https://www.digikey.com/en/products/detail/abracon-llc/AOTA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 -> https://www.lcsc.com/product-detail/C42411119.html
- L2: Link (none) -> https://www.lcsc.com/product-detail/C435392.html
- Q1: Link (none) -> https://www.lcsc.com/product-detail/C7420322.html
- R1, R10, R4, R7: Link (none) -> https://www.lcsc.com/product-detail/C2930092.html
- R11, R12, R2, R3, R5, R6, R8, R9: Link (none) -> https://www.lcsc.com/product-detail/C2907020.html
- R13, R19, R22, R23, R24: Link (none) -> https://www.lcsc.com/product-detail/C2906868.html
- R14, R15: Link (none) -> https://www.lcsc.com/product-detail/C2906982.html
- R16: Link (none) -> https://www.lcsc.com/product-detail/C2906979.html
- R17, R18: value 100k -> 10k; Link (none) -> https://www.lcsc.com/product-detail/C2906868.html
- R20: Link (none) -> https://www.lcsc.com/product-detail/C48533697.html
- R21: Link (none) -> https://www.lcsc.com/product-detail/C2909352.html
- R25: Link (none) -> https://www.lcsc.com/product-detail/C2906864.html
- R26, R27: Link (none) -> https://www.lcsc.com/product-detail/C2909343.html
- R28, R29, R30, R34: Link (none) -> https://www.lcsc.com/product-detail/C2907002.html
- TP1: now left out of the parts list
- U2: Link (none) -> https://www.lcsc.com/product-detail/C42267816.html
- U3: Link (none) -> https://www.lcsc.com/product-detail/C528622.html
- U6: Link (none) -> https://www.lcsc.com/product-detail/C5354566.html
- U7: Link (none) -> https://www.lcsc.com/product-detail/C41408446.html
Connections:
- net GND_CORE: now also C37.2
- net at D1.1 (K), D2.1 (K), D4.1 (K)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: now also C37.1
Other:
- moved on the sheet: BT1, C25, C26, C36, C4, C5, C7, C8, D1, D10, D11, D12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
