File: hardware/TileGlobeMC_Node/TileGlobeMC_Node.kicad_pcb (KiCad board)
At the start: 2 copper layers, 36 x 36 mm, 76 parts, among them J10 LCD, J9 SWD, Q1 2N7002, Q2 2N7002, U1 RP2350_80QFN, U2 TPS62A01DRL, U3 BQ24232RGT, U4 ESP-PSRAM64H, U5 PY25Q128HA-WXH, U6 PY25Q128HA-SSH, U7 74AHC1G04, U8 74AHC1G32, Y1 12M

Commit message: Commit before switching to multi board design
Parts:
- added C29: 100n, Capacitor_SMD:C_0402_1005Metric, F.Cu at (-24.0, 24.5)
- added C30: 100n, Capacitor_SMD:C_0402_1005Metric, F.Cu at (-24.0, 26.5)
- added C31: 100n, Capacitor_SMD:C_0402_1005Metric, F.Cu at (-24.0, 28.4)
- added C32: 100n, Capacitor_SMD:C_0402_1005Metric, F.Cu at (-24.0, 30.4)
- added C33: 100n, Capacitor_SMD:C_0402_1005Metric, F.Cu at (-21.2, 24.5)
- added C34: 100n, Capacitor_SMD:C_0402_1005Metric, F.Cu at (-21.2, 26.5)
- added D1: 1N4148WT, Diode_SMD:D_SOD-523, F.Cu at (-23.7, 12.5)
- added D2: 1N4148WT, Diode_SMD:D_SOD-523, F.Cu at (-23.7, 14.9)
- added D3: 3V, Diode_SMD:D_SOD-523, F.Cu at (-23.7, 17.4)
- added D4: 1N4148WT, Diode_SMD:D_SOD-523, F.Cu at (-23.7, 19.9)
- added D5: 3V, Diode_SMD:D_SOD-523, F.Cu at (-23.7, 22.3)
- added R32: 5.1k, Capacitor_SMD:C_0402_1005Metric, F.Cu at (-21.2, 28.4)
- added R33: 5.1k, Capacitor_SMD:C_0402_1005Metric, F.Cu at (-21.2, 30.4)
- added R34: 100k, Capacitor_SMD:C_0402_1005Metric, F.Cu at (-18.3, 24.5)
- added R35: 10k, Capacitor_SMD:C_0402_1005Metric, F.Cu at (-18.3, 26.5)
- added R36: 10k, Capacitor_SMD:C_0402_1005Metric, F.Cu at (-18.3, 28.4)
- added R37: 10k, Capacitor_SMD:C_0402_1005Metric, F.Cu at (-18.3, 30.4)
- added R38: 10k, Capacitor_SMD:C_0402_1005Metric, F.Cu at (-15.4, 24.5)
- added R39: 10k, Capacitor_SMD:C_0402_1005Metric, F.Cu at (-15.4, 26.5)
- added R40: 10k, Capacitor_SMD:C_0402_1005Metric, F.Cu at (-15.4, 28.4)
- added R41: 10k, Capacitor_SMD:C_0402_1005Metric, F.Cu at (-15.4, 30.4)
- added SW1: Left, Button_Switch_SMD:SW_SPST_PTS647_Sx38, B.Cu at (0.00, 0.00)
- added SW2: Left, Button_Switch_SMD:SW_SPST_PTS647_Sx38, B.Cu at (13.0, 0.00)
- added SW3: Left, Button_Switch_SMD:SW_SPST_PTS647_Sx38, B.Cu at (0.00, 13.0)
- added SW4: Left, Button_Switch_SMD:SW_SPST_PTS647_Sx38, B.Cu at (-13.0, 0.00)
- added SW5: Left, Button_Switch_SMD:SW_SPST_PTS647_Sx38, B.Cu at (0.00, -13.0)
- J10: moved to B.Cu
- U8: value 74AHC1G32 -> SC7A20; footprint Package_TO_SOT_SMD:SOT-23-5 -> Package_LGA:LGA-12_2x2mm_P0.5mm
- moved U8 62.3 mm to (-23.5, 33.4)
- moved U5 35.8 mm to (19.7, -25.5), turned to 90 degrees
- moved U6 25.9 mm to (19.7, -25.5), turned to 90 degrees
- moved U4 19.2 mm to (30.3, -20.9)
- moved C10 10.7 mm to (32.2, 27.0)
- moved C11 10.7 mm to (32.2, 29.0)
- moved C2 10.7 mm to (32.7, 11.1)
- moved C22 10.7 mm to (38.2, 8.38)
- moved C24 10.7 mm to (38.0, 13.7)
- moved C3 10.7 mm to (32.2, 13.7)
- moved C4 10.7 mm to (32.2, 17.1)
- moved C5 10.7 mm to (32.2, 19.1)
- moved C6 10.7 mm to (32.2, 21.1)
- moved C7 10.7 mm to (32.2, 23.1)
- moved C9 10.7 mm to (32.2, 25.0)
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Connections:
- net BAT_ISET_SAMPLE renamed BAT_ICHG_SAMPLE
- net VIN_~{PGOOD} renamed Net-(U3-PGOOD)
- R23 pad 2: unconnected-(R23-Pad2) -> Net-(D5-K)
- U2 pad 4: 3V3_EN -> Net-(D1-K)
- U8 pad 1: 3V3_EN_LATCH -> unconnected-(U8-SDO-Pad1)
- U8 pad 2: VIN_PGOOD -> I2C_SDA
- U8 pad 3: GND -> +3V3
- U8 pad 4: 3V3_EN -> GND
- U8 pad 5: VBUS -> unconnected-(U8-INT1-Pad5)
Other:
- board outline removed

Commit message: PCB progress
Parts:
- removed Q2: 2N7002, Package_TO_SOT_SMD:SOT-23
- removed U5: PY25Q128HA-WXH, Package_SON:WSON-8-1EP_6x5mm_P1.27mm_EP3.4x4.3mm
- added BT1: LIR2450, Project:BS-24-B___014, B.Cu at (0.00, 0.00)
- added C35: 100n, Capacitor_SMD:C_0603_1608Metric, F.Cu at (87.8, -28.1)
- added C36: 120p, Capacitor_SMD:C_0402_1005Metric, F.Cu at (7.38, 9.53)
- added D10: ESD5Z3.3C, Diode_SMD:D_SOD-523, B.Cu at (-16.7, 9.20)
- added D11: ESD5Z3.3C, Diode_SMD:D_SOD-523, B.Cu at (-16.7, 11.7)
- added D12: ESD5Z3.3C, Diode_SMD:D_SOD-523, B.Cu at (16.7, 11.7)
- added D13: ESD5Z3.3C, Diode_SMD:D_SOD-523, B.Cu at (16.7, 9.20)
- added D14: ESD5Z3.3C, Diode_SMD:D_SOD-523, B.Cu at (16.7, 6.70)
- added D15: ESD5Z3.3C, Diode_SMD:D_SOD-523, B.Cu at (16.7, -6.70)
- added D16: ESD5Z3.3C, Diode_SMD:D_SOD-523, B.Cu at (16.7, -9.20)
- added D17: ESD5Z3.3C, Diode_SMD:D_SOD-523, B.Cu at (16.7, -11.7)
- added D18: ESD5Z3.3C, Diode_SMD:D_SOD-523, B.Cu at (-11.7, 16.7)
- added D19: ESD5Z3.3C, Diode_SMD:D_SOD-523, B.Cu at (-9.20, 16.7)
- added D20: ESD5Z3.3C, Diode_SMD:D_SOD-523, B.Cu at (-6.70, 16.7)
- added D21: ESD5Z3.3C, Diode_SMD:D_SOD-523, B.Cu at (6.70, 16.7)
- added D22: ESD5Z3.3C, Diode_SMD:D_SOD-523, B.Cu at (9.20, 16.7)
- added D23: ESD5Z3.3C, Diode_SMD:D_SOD-523, B.Cu at (11.7, 16.7)
- added D24: ESD5Z3.3C, Diode_SMD:D_SOD-523, B.Cu at (11.7, -16.7)
- added D25: ESD5Z3.3C, Diode_SMD:D_SOD-523, B.Cu at (9.20, -16.7)
- added D26: ESD5Z3.3C, Diode_SMD:D_SOD-523, B.Cu at (6.70, -16.7)
- added D27: ESD5Z3.3C, Diode_SMD:D_SOD-523, B.Cu at (-6.70, -16.7)
- added D28: ESD5Z3.3C, Diode_SMD:D_SOD-523, B.Cu at (-9.20, -16.7)
- added D29: ESD5Z3.3C, Diode_SMD:D_SOD-523, B.Cu at (-11.7, -16.7)
- added D6: ESD5Z3.3C, Diode_SMD:D_SOD-523, B.Cu at (-16.7, -11.7)
- added D7: ESD5Z3.3C, Diode_SMD:D_SOD-523, B.Cu at (-16.7, -9.20)
- added D8: ESD5Z3.3C, Diode_SMD:D_SOD-523, B.Cu at (-16.7, -6.70)
- added D9: ESD5Z3.3C, Diode_SMD:D_SOD-523, B.Cu at (-16.7, 6.70)
- added H1: MountingHole, MountingHole:MountingHole_2.2mm_M2, F.Cu at (-17.8, -17.8)
- added H2: MountingHole, MountingHole:MountingHole_2.2mm_M2, F.Cu at (-17.8, 17.8)
- added H3: MountingHole, MountingHole:MountingHole_2.2mm_M2, F.Cu at (17.8, 17.8)
- added H4: MountingHole, MountingHole:MountingHole_2.2mm_M2, F.Cu at (17.8, -17.8)
- added H5: MountingHole, MountingHole:MountingHole_2.2mm_M2, F.Cu at (28.2, -17.8)
- added H6: MountingHole, MountingHole:MountingHole_2.2mm_M2, F.Cu at (28.2, 17.8)
- added H7: MountingHole, MountingHole:MountingHole_2.2mm_M2, F.Cu at (63.8, 17.8)
- added H8: MountingHole, MountingHole:MountingHole_2.2mm_M2, F.Cu at (63.8, -17.8)
- added J1: P_Female, Project:BC-20-5PD160, F.Cu at (-20.0, 8.00)
- added J11: USB_C, Connector_USB:USB_C_Receptacle_GCT_USB4105-xx-A_16P_TopMnt_Horizontal, B.Cu at (62.3, 0.10)
- added J12: P_Female_Fallback, Project:PinSocket_1x05_P2.54mm_Horizontal_NoSilk, F.Cu at (-15.5, 2.92)
- added J13: P_Male_Fallback, Project:PinHeader_1x05_P2.54mm_Horizontal_NoSilk, F.Cu at (-15.5, -2.92)
- added J14: P_Female_Fallback, Project:PinSocket_1x05_P2.54mm_Horizontal_NoSilk, F.Cu at (15.5, -2.92)
- added J15: P_Male_Fallback, Project:PinHeader_1x05_P2.54mm_Horizontal_NoSilk, F.Cu at (15.5, 2.92)
- added J16: P_Female_Fallback, Project:PinSocket_1x05_P2.54mm_Horizontal_NoSilk, F.Cu at (2.92, 15.5)
- added J17: P_Male_Fallback, Project:PinHeader_1x05_P2.54mm_Horizontal_NoSilk, F.Cu at (-2.92, 15.5)
- added J18: P_Female_Fallback, Project:PinSocket_1x05_P2.54mm_Horizontal_NoSilk, F.Cu at (-2.92, -15.5)
- added J19: P_Male_Fallback, Project:PinHeader_1x05_P2.54mm_Horizontal_NoSilk, F.Cu at (2.92, -15.5)
- added J2: P_Male, Project:BC-15-5P380, F.Cu at (-20.0, -8.00)
- added J20: Conn_01x24_MountingPin, Project:FPC_Verticle_24pin_0.5mm, F.Cu at (10.0, 0.00)
- added J3: P_Female, Project:BC-20-5PD160, F.Cu at (8.00, 20.0)
- added J4: P_Male, Project:BC-15-5P380, F.Cu at (-8.00, 20.0)
- added J5: P_Female, Project:BC-20-5PD160, F.Cu at (20.0, -8.00)
- added J6: P_Male, Project:BC-15-5P380, F.Cu at (20.0, 8.00)
- added J7: P_Female, Project:BC-20-5PD160, F.Cu at (-8.00, -20.0)
- added J8: P_Male, Project:BC-15-5P380, F.Cu at (8.00, -20.0)
- added JP3: BL_P1_1, Jumper:SolderJumper-2_P1.3mm_Open_TrianglePad1.0x1.5mm, F.Cu at (96.0, -30.1)
- added JP4: BL_P1_2, Jumper:SolderJumper-2_P1.3mm_Open_TrianglePad1.0x1.5mm, F.Cu at (96.0, -26.5)
- added JP5: BL_P1_3, Jumper:SolderJumper-2_P1.3mm_Open_TrianglePad1.0x1.5mm, F.Cu at (96.0, -23.0)
- added R42: 100k, Resistor_SMD:R_0603_1608Metric, F.Cu at (91.8, -28.1)
- added R43: 100k, Resistor_SMD:R_0603_1608Metric, F.Cu at (91.8, -25.6)
- added R44: 100k, Resistor_SMD:R_0603_1608Metric, F.Cu at (91.8, -23.1)
- added R45: 100k, Resistor_SMD:R_0603_1608Metric, F.Cu at (91.8, -20.5)
- added R46: 100k, Resistor_SMD:R_0603_1608Metric, F.Cu at (91.8, -18.0)
- added R47: 100k, Resistor_SMD:R_0603_1608Metric, F.Cu at (91.8, -15.5)
- added U9: AW9523B, Package_DFN_QFN:QFN-24-1EP_4x4mm_P0.5mm_EP2.7x2.7mm, F.Cu at (85.3, -3.40)
- C27, C28, C29, C30, C31, C32, C33, C34, C4, C5, C6, C7: footprint Capacitor_SMD:C_0402_1005Metric -> Capacitor_SMD:C_0603_1608Metric
- J9: moved to B.Cu
- JP1: footprint TestPoint:TestPoint_2Pads_Pitch2.54mm_Drill0.8mm -> Connector_PinHeader_1.00mm:PinHeader_1x02_P1.00mm_Vertical
- JP2: footprint TestPoint:TestPoint_2Pads_Pitch2.54mm_Drill0.8mm -> Connector_PinHeader_1.00mm:PinHeader_1x02_P1.00mm_Vertical; moved to B.Cu
- R1, R14, R17, R18, R19, R2, R22, R23, R26, R27, R3, R32, R33, R34, R35, R36, R37, R38, R39, R4, R40, R41, R5, R6, R8, R9: footprint Capacitor_SMD:C_0402_1005Metric -> Resistor_SMD:R_0603_1608Metric
- R10, R11, R12, R28, R29, R30, R7: footprint Capacitor_SMD:C_0402_1005Metric -> Resistor_SMD:R_0603_1608Metric; moved to B.Cu
- R13, R20, R21, R24, R25: footprint Capacitor_SMD:C_0402_1005Metric -> Resistor_SMD:R_0402_1005Metric
- R15: value 17.4k -> 10k; footprint Capacitor_SMD:C_0402_1005Metric -> Resistor_SMD:R_0603_1608Metric
- R16: value 1.5k -> 1.8k; footprint Capacitor_SMD:C_0402_1005Metric -> Resistor_SMD:R_0603_1608Metric
- R31: value 4.7 -> 100k; footprint Capacitor_SMD:C_0402_1005Metric -> Resistor_SMD:R_0603_1608Metric
- SW1, SW2, SW3, SW4, SW5: moved to F.Cu
- U2: value TPS62A01DRL -> TPS62A01PDDC; footprint Package_TO_SOT_SMD:SOT-563 -> Package_TO_SOT_SMD:SOT-23-6
- U8: value SC7A20 -> LSM6DS3; footprint Package_LGA:LGA-12_2x2mm_P0.5mm -> Package_LGA:LGA-14_3x2.5mm_P0.5mm_LayoutBorder3x4y
- moved U8 125.5 mm to (96.2, -4.53)
- moved R41 123.4 mm to (91.8, -30.6)
- moved C34 123.0 mm to (87.8, -30.6)
- moved D3 122.5 mm to (95.5, -10.9)
- moved C29 118.9 mm to (83.8, -25.6)
- moved C30 118.6 mm to (83.8, -23.1)
- moved C31 118.4 mm to (83.8, -20.5)
- moved C32 118.2 mm to (83.8, -18.0)
- moved R19 118.1 mm to (-74.3, 25.0), turned to 90 degrees
- moved R35 117.1 mm to (87.8, -23.1)
- moved R38 112.6 mm to (87.8, -20.5)
- moved R39 112.4 mm to (87.8, -18.0)
- moved C33 112.3 mm to (83.8, -15.5)
- moved R40 112.2 mm to (87.8, -15.5)
- moved R17 111.9 mm to (-67.9, 25.1)
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Connections:
- net /RP_VREG_LX renamed /Core/RP_VREG_LX
- net /SWCLK renamed /Core/SWCLK
- net /SWD renamed /Core/SWD
- net BTN_CENTER renamed /Peripheral/BTN_CENTER
- net LCD_CS renamed /Peripheral/LCD_CS
- net LCD_DC renamed /Peripheral/LCD_DC
- net LCD_SCL renamed /Peripheral/LCD_SCK
- net LCD_SDA renamed /Peripheral/LCD_MOSI
- net USB_D+ renamed /Core/USB_D+
- net USB_D- renamed /Core/USB_D-
- net VIN renamed /Core/VIN
- C1 pad 2: GND -> GND_CORE
- C10 pad 2: GND -> GND_CORE
- C11 pad 2: GND -> GND_CORE
- C12 pad 2: GND -> GND_CORE
- C13 pad 2: GND -> GND_CORE
- C14 pad 2: GND -> GND_CORE
- C15 pad 2: GND -> GND_CORE
- C16 pad 2: GND -> GND_CORE
- C17 pad 2: GND -> GND_CORE
- C18 pad 2: GND -> GND_CORE
- C19 pad 2: GND -> GND_CORE
- C2 pad 2: GND -> GND_CORE
- C20 pad 2: GND -> GND_CORE
- C21 pad 2: GND -> GND_CORE
- C22 pad 2: GND -> GND_CORE
- C23 pad 1: GND -> GND_CORE
- C24 pad 1: GND -> GND_CORE
- C25 pad 2: GND -> GND_CORE
- C26 pad 2: GND -> GND_CORE
- C27 pad 1: +3V3 -> /Peripheral/+3V3
- C27 pad 2: GND -> GND_PERI
- C28 pad 1: +3V3 -> /Peripheral/+3V3
- C28 pad 2: GND -> GND_PERI
- C29 pad 1: +3V3 -> /Peripheral/+3V3
- C29 pad 2: GND -> GND_PERI
- C3 pad 2: GND -> GND_CORE
- C30 pad 2: GND -> GND_PERI
- C31 pad 2: GND -> GND_PERI
- C32 pad 2: GND -> GND_PERI
- C33 pad 2: GND -> GND_PERI
- C34 pad 2: GND -> GND_PERI
- C4 pad 2: GND -> GND_CORE
- C5 pad 2: GND -> GND_CORE
- C6 pad 1: GND -> GND_CORE
- C7 pad 2: GND -> GND_CORE
- C8 pad 2: GND -> GND_CORE
- C9 pad 2: GND -> GND_CORE
- D1 pad 2: BTN_CENTER_VBUS -> /Core/BTN_CENTER_VBUS
- D3 pad 2: GND -> GND_PERI
- D5 pad 2: GND -> GND_CORE
- J10 pad 1: GND -> GND_PERI
- J10 pad 12: GND -> GND_PERI
- J10 pad 2: Net-(J10-Pin_2) -> LCD_BL
- J10 pad 3: +3V3 -> /Peripheral/+3V3
- J10 pad 4: +3V3 -> /Peripheral/+3V3
- J10 pad 5: GND -> GND_PERI
- J10 pad 6: GND -> GND_PERI
- J10 pad MP: GND -> GND_PERI
- J9 pad 2: GND -> GND_CORE
- J9 pad MP: GND -> GND_CORE
- JP1 pad 1: GND -> GND_CORE
- JP2 pad 1: GND -> GND_CORE
- Q1 pad 2: GND -> GND_CORE
- R1 pad 1: /PA.CAR -> /Core/PA.CAR
- R1 pad 2: /PA.CA -> /Core/PA.CA
- R10 pad 1: /PD.CAR -> /Core/PD.CAR
- R10 pad 2: /PD.CA -> /Core/PD.CA
- R11 pad 2: /PD.D1 -> /Core/PD.D1
- R12 pad 2: /PD.D3 -> /Core/PD.D3
- R14 pad 1: GND -> GND_CORE
- R15 pad 1: GND -> GND_CORE
- R16 pad 2: GND -> GND_CORE
- R19 pad 1: GND -> GND_CORE
- R2 pad 2: /PA.D1 -> /Core/PA.D1
- R20 pad 1: GND -> GND_CORE
- R3 pad 2: /PA.D3 -> /Core/PA.D3
- R31 pad 1: Net-(Q2-D) -> BTN_LEFT
- R31 pad 2: Net-(J10-Pin_2) -> GND_PERI
- R32 pad 1: GND -> GND_PERI
- R33 pad 1: GND -> GND_PERI
- R34 pad 1: GND -> GND_CORE
- R35 pad 1: BTN_CENTER_VBUS -> /Peripheral/BTN_CENTER_VBUS
- R36 pad 1: unconnected-(R36-Pad1) -> /Peripheral/I2C_SCL
- R36 pad 2: +3V3 -> /Peripheral/+3V3
- R37 pad 1: unconnected-(R37-Pad1) -> /Peripheral/I2C_SDA
- R37 pad 2: +3V3 -> /Peripheral/+3V3
- R4 pad 1: /PB.CAR -> /Core/PB.CAR
- R4 pad 2: /PB.CA -> /Core/PB.CA
- R5 pad 2: /PB.D1 -> /Core/PB.D1
- R6 pad 2: /PB.D3 -> /Core/PB.D3
- R7 pad 1: /PC.CAR -> /Core/PC.CAR
- R7 pad 2: /PC.CA -> /Core/PC.CA
- R8 pad 2: /PC.D1 -> /Core/PC.D1
- R9 pad 2: /PC.D3 -> /Core/PC.D3
- SW1 pad 1: BTN_CENTER_VBUS -> /Peripheral/BTN_CENTER_VBUS
- SW1 pad 2: VBUS -> /Peripheral/VBUS_1
- SW2 pad 2: +3V3 -> /Peripheral/+3V3
- SW3 pad 2: +3V3 -> /Peripheral/+3V3
- SW4 pad 2: +3V3 -> /Peripheral/+3V3
- SW5 pad 2: +3V3 -> /Peripheral/+3V3
- U1 pad 1: unconnected-(U1-GPIO4-Pad1) -> /Core/PD.D1
- U1 pad 11: unconnected-(U1-GPIO12-Pad11) -> /Core/PA.D2
- U1 pad 12: unconnected-(U1-GPIO13-Pad12) -> /Core/PA.D3
- U1 pad 13: unconnected-(U1-GPIO14-Pad13) -> /Core/PA.CB
- U1 pad 14: unconnected-(U1-GPIO15-Pad14) -> /Core/PB.CAR
- U1 pad 16: unconnected-(U1-GPIO16-Pad16) -> /Core/PB.CA
- U1 pad 17: unconnected-(U1-GPIO17-Pad17) -> /Core/PB.D0
- U1 pad 18: unconnected-(U1-GPIO18-Pad18) -> /Core/PB.D1
- U1 pad 19: unconnected-(U1-GPIO19-Pad19) -> /Core/PB.D2
- U1 pad 2: unconnected-(U1-GPIO5-Pad2) -> /Core/PD.D2
- U1 pad 20: unconnected-(U1-GPIO20-Pad20) -> /Core/PB.D3
- U1 pad 21: unconnected-(U1-GPIO21-Pad21) -> /Core/PB.CB
- U1 pad 22: unconnected-(U1-GPIO22-Pad22) -> /Core/PC.CAR
- U1 pad 23: unconnected-(U1-GPIO23-Pad23) -> /Core/PC.CA
- U1 pad 25: unconnected-(U1-GPIO24-Pad25) -> /Core/PC.D0
- U1 pad 26: unconnected-(U1-GPIO25-Pad26) -> /Core/PC.D1
- U1 pad 27: unconnected-(U1-GPIO26-Pad27) -> /Core/PC.D2
- U1 pad 28: unconnected-(U1-GPIO27-Pad28) -> /Core/PC.D3
- U1 pad 3: unconnected-(U1-GPIO6-Pad3) -> /Core/PD.D3
- U1 pad 36: unconnected-(U1-GPIO28-Pad36) -> /Core/PC.CB
- U1 pad 37: unconnected-(U1-GPIO29-Pad37) -> 3V3_EN_LATCH
- U1 pad 38: unconnected-(U1-GPIO30-Pad38) -> BAT_~{CHG}
- U1 pad 39: unconnected-(U1-GPIO31-Pad39) -> BAT_SAMPLE_EN
- U1 pad 4: unconnected-(U1-GPIO7-Pad4) -> /Core/PD.CB
- U1 pad 40: unconnected-(U1-GPIO32-Pad40) -> Net-(D5-K)
- U1 pad 42: unconnected-(U1-GPIO33-Pad42) -> /Core/GPIO0
- U1 pad 43: unconnected-(U1-GPIO34-Pad43) -> /Core/GPIO1
- U1 pad 44: unconnected-(U1-GPIO35-Pad44) -> /Core/GPIO2
- U1 pad 45: unconnected-(U1-GPIO36-Pad45) -> /Core/GPIO3
- U1 pad 46: unconnected-(U1-GPIO37-Pad46) -> /Core/GPIO4
- U1 pad 47: unconnected-(U1-GPIO38-Pad47) -> /Core/GPIO5
- U1 pad 48: unconnected-(U1-GPIO39-Pad48) -> /Core/GPIO6
- U1 pad 49: unconnected-(U1-GPIO40_ADC0-Pad49) -> /Core/GPIO7
- U1 pad 52: unconnected-(U1-GPIO41_ADC1-Pad52) -> /Core/GPIO8
- U1 pad 53: unconnected-(U1-GPIO42_ADC2-Pad53) -> /Core/GPIO9
- U1 pad 54: unconnected-(U1-GPIO43_ADC3-Pad54) -> /Core/GPIO10
- U1 pad 55: unconnected-(U1-GPIO44_ADC4-Pad55) -> /Core/GPIO11
- U1 pad 56: unconnected-(U1-GPIO45_ADC5-Pad56) -> /Core/GPIO12
- U1 pad 57: unconnected-(U1-GPIO46_ADC6-Pad57) -> BAT_ICHG_SAMPLE
- U1 pad 58: unconnected-(U1-GPIO47_ADC7-Pad58) -> BAT_SAMPLE
- U1 pad 6: unconnected-(U1-GPIO8-Pad6) -> /Core/PA.CAR
- U1 pad 62: GND -> GND_CORE
- U1 pad 7: unconnected-(U1-GPIO9-Pad7) -> /Core/PA.CA
- U1 pad 78: unconnected-(U1-GPIO1-Pad78) -> /Core/PD.CAR
- U1 pad 79: unconnected-(U1-GPIO2-Pad79) -> /Core/PD.CA
- U1 pad 8: unconnected-(U1-GPIO10-Pad8) -> /Core/PA.D0
- U1 pad 80: unconnected-(U1-GPIO3-Pad80) -> /Core/PD.D0
- U1 pad 81: GND -> GND_CORE
- U1 pad 9: unconnected-(U1-GPIO11-Pad9) -> /Core/PA.D1
- U2 pad 1: GND -> Net-(D1-K)
- U2 pad 2: Net-(U2-SW) -> GND_CORE
- U2 pad 3: VBUS -> Net-(U2-SW)
- U2 pad 4: Net-(D1-K) -> VBUS
- U2 pad 5: Net-(U2-FB) -> unconnected-(U2-PG-Pad5)
- U2 pad 6: unconnected-(U2-PG-Pad6) -> Net-(U2-FB)
- U3 pad 17: GND -> GND_CORE
- U3 pad 4: GND -> GND_CORE
- U3 pad 5: GND -> GND_CORE
- U3 pad 8: GND -> GND_CORE
- U4 pad 4: GND -> GND_CORE
- U6 pad 4: GND -> GND_CORE
- U7 pad 3: GND -> GND_CORE
- U8 pad 1: unconnected-(U8-SDO-Pad1) -> GND_PERI
- U8 pad 12: I2C_SCL -> /Peripheral/+3V3
- U8 pad 2: I2C_SDA -> GND_PERI
- U8 pad 3: +3V3 -> GND_PERI
- U8 pad 4: GND -> IMU_INT1
- U8 pad 5: unconnected-(U8-INT1-Pad5) -> /Peripheral/+3V3
- U8 pad 6: unconnected-(U8-INT2-Pad6) -> GND_PERI
- U8 pad 7: +3V3 -> GND_PERI
- U8 pad 8: GND -> /Peripheral/+3V3
- U8 pad 9: GND -> IMU_INT2
- Y1 pad 2: GND -> GND_CORE
- Y1 pad 4: GND -> GND_CORE
Routing:
- net GND_CORE: track 0.00 -> 94.5 mm, vias 0 -> 2
- net (no net): track 0.00 -> 46.9 mm, vias 0 -> 12
- net /Core/PD.D2: track 0.00 -> 29.0 mm, vias 0 -> 1
- net /Core/PD.CAR: track 0.00 -> 25.7 mm, vias 0 -> 1
- net /Core/PD.D0: track 0.00 -> 23.8 mm, vias 0 -> 1
- net RP_DVDD: track 0.00 -> 22.6 mm, vias 0 -> 9
- net /Core/PD.CA: track 0.00 -> 21.6 mm, vias 0 -> 1
- net /Core/PD.D3: track 0.00 -> 21.6 mm, vias 0 -> 1
- net /Core/PD.D1: track 0.00 -> 20.7 mm, vias 0 -> 1
- net /Core/PA.CB: track 0.00 -> 20.7 mm
- net +3V3: track 0.00 -> 19.0 mm, vias 0 -> 10
- net /Core/PA.CAR: track 0.00 -> 18.3 mm
- net QMI_SCK: track 0.00 -> 18.2 mm
- net QMI_SD0: track 0.00 -> 17.9 mm
- net QMI_SD3: track 0.00 -> 17.8 mm
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- added copper zone on F.Cu, net /Core/RP_VREG_LX
- added copper zone on F.Cu, net GND_CORE
- added copper zone on F.Cu, net RP_DVDD
Other:
- board outline added: 86 x 40 mm
- copper layers 2 -> 4

Commit message: Main PCB progress
Parts:
- removed JP1: RESET, Connector_PinHeader_1.00mm:PinHeader_1x02_P1.00mm_Vertical
- added J21: Conn_01x24_MountingPin, Project:FPC_Verticle_24pin_0.5mm, F.Cu at (62.1, -26.7)
- added TP1: RP_RUN, TestPoint:TestPoint_THTPad_D1.0mm_Drill0.5mm, F.Cu at (3.15, 7.55)
- Q1: value 2N7002 -> 2N7002W; footprint Package_TO_SOT_SMD:SOT-23 -> Package_TO_SOT_SMD:SOT-323_SC-70
- R17, R18, R19, R22, R23, R26, R27: footprint Resistor_SMD:R_0603_1608Metric -> Resistor_SMD:R_0402_1005Metric
- R34, R8: moved to B.Cu
- U1: footprint RP2350:RP2350-QFN-80-1EP_10x10_P0.4mm_EP3.4x3.4mm_ThermalVias -> Project:RP2350-QFN-80-1EP_10x10_P0.4mm_EP3.4x3.4mm_ThermalVias
- U3: footprint Package_DFN_QFN:VQFN-16-1EP_3x3mm_P0.5mm_EP1.68x1.68mm_ThermalVias -> Project:VQFN-16-1EP_3x3mm_P0.5mm_EP1.68x1.68mm_ThermalVias
- U7: footprint Package_TO_SOT_SMD:SOT-23-5 -> Package_TO_SOT_SMD:SOT-353_SC-70-5
- moved R19 90.9 mm to (9.60, -10.0), turned to -90 degrees
- moved Q1 86.3 mm to (7.42, -10.0), turned to 180 degrees
- moved R17 82.0 mm to (7.22, -7.78), turned to -90 degrees
- moved R18 78.3 mm to (6.28, -7.78), turned to 90 degrees
- moved R23 55.1 mm to (5.25, 8.45)
- moved D5 52.4 mm to (5.55, 7.25)
- moved R26 37.7 mm to (6.75, -5.35)
- moved D1 36.1 mm to (7.95, 7.40), turned to 90 degrees
- moved D2 34.8 mm to (7.55, 12.2), turned to 180 degrees
- moved R27 34.4 mm to (6.75, -6.30)
- moved R22 32.1 mm to (4.15, 12.2), turned to 0 degrees
- moved U7 30.3 mm to (4.55, 10.3), turned to 180 degrees
- moved R34 27.7 mm to (9.78, 12.9), turned to 180 degrees
- moved R6 4.71 mm to (3.70, 13.8)
- moved JP2 1.14 mm to (-13.2, -7.31)
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Connections:
- J11 pad A4: /Peripheral/VIN_1 -> /Peripheral/VIN
- J11 pad B4: /Peripheral/VIN_2 -> /Peripheral/VIN
- J11 pad B9: /Peripheral/VIN_3 -> /Peripheral/VIN
- J20 pad 1: unconnected-(J20-Pin_1-Pad1) -> GND_CORE
- J20 pad 10: unconnected-(J20-Pin_10-Pad10) -> /Core/GPIO9
- J20 pad 11: unconnected-(J20-Pin_11-Pad11) -> /Core/GPIO8
- J20 pad 12: unconnected-(J20-Pin_12-Pad12) -> /Core/GPIO7
- J20 pad 13: unconnected-(J20-Pin_13-Pad13) -> /Core/GPIO6
- J20 pad 14: unconnected-(J20-Pin_14-Pad14) -> /Core/GPIO5
- J20 pad 15: unconnected-(J20-Pin_15-Pad15) -> /Core/GPIO4
- J20 pad 16: unconnected-(J20-Pin_16-Pad16) -> /Core/GPIO3
- J20 pad 17: unconnected-(J20-Pin_17-Pad17) -> /Core/GPIO2
- J20 pad 18: unconnected-(J20-Pin_18-Pad18) -> /Core/GPIO1
- J20 pad 19: unconnected-(J20-Pin_19-Pad19) -> /Core/GPIO0
- J20 pad 2: unconnected-(J20-Pin_2-Pad2) -> /Core/USB_D-
- J20 pad 20: unconnected-(J20-Pin_20-Pad20) -> /Core/VIN
- J20 pad 21: unconnected-(J20-Pin_21-Pad21) -> /Core/VIN
- J20 pad 22: unconnected-(J20-Pin_22-Pad22) -> VBUS
- J20 pad 23: unconnected-(J20-Pin_23-Pad23) -> /Core/BTN_CENTER_VBUS
- J20 pad 24: unconnected-(J20-Pin_24-Pad24) -> GND_CORE
- J20 pad 3: unconnected-(J20-Pin_3-Pad3) -> /Core/USB_D+
- J20 pad 7: unconnected-(J20-Pin_7-Pad7) -> /Core/GPIO12
- J20 pad 8: unconnected-(J20-Pin_8-Pad8) -> /Core/GPIO11
- J20 pad 9: unconnected-(J20-Pin_9-Pad9) -> /Core/GPIO10
- J20 pad MP: unconnected-(J20-MountPin-PadMP) -> GND_CORE
- J9 pad MP: GND_CORE -> /Core/VIN
- SW1 pad 2: /Peripheral/VBUS_1 -> /Peripheral/VBUS
- U1 pad 14: /Core/PB.CAR -> BAT_~{CHG}
- U1 pad 16: /Core/PB.CA -> /Core/PB.CAR
- U1 pad 17: /Core/PB.D0 -> /Core/PB.CA
- U1 pad 18: /Core/PB.D1 -> /Core/PB.D0
- U1 pad 19: /Core/PB.D2 -> /Core/PB.D1
- U1 pad 20: /Core/PB.D3 -> /Core/PB.D2
- U1 pad 21: /Core/PB.CB -> /Core/PB.D3
- U1 pad 22: /Core/PC.CAR -> /Core/PB.CB
- U1 pad 23: /Core/PC.CA -> 3V3_EN_LATCH
- U1 pad 25: /Core/PC.D0 -> /Core/PC.CAR
- U1 pad 26: /Core/PC.D1 -> /Core/PC.CA
- U1 pad 27: /Core/PC.D2 -> /Core/PC.D0
- U1 pad 28: /Core/PC.D3 -> /Core/PC.D1
- U1 pad 36: /Core/PC.CB -> /Core/PC.D2
- U1 pad 37: 3V3_EN_LATCH -> /Core/PC.D3
- U1 pad 38: BAT_~{CHG} -> /Core/PC.CB
- U1 pad 39: BAT_SAMPLE_EN -> Net-(D5-K)
- U1 pad 40: Net-(D5-K) -> BAT_SAMPLE_EN
Routing:
- net /Core/VIN: track 14.3 -> 182.5 mm, vias 1 -> 4
- net +3V3: track 19.0 -> 105.7 mm, vias 10 -> 9
- net +BATT: track 5.30 -> 41.4 mm, vias 1 -> 4
- net VBUS: track 3.50 -> 35.8 mm, vias 1 -> 4
- net GND_CORE: track 94.5 -> 126.2 mm, vias 2 -> 34
- net BAT_ICHG_SAMPLE: track 1.88 -> 30.3 mm, vias 0 -> 2
- net /Core/PC.CB: track 3.91 -> 31.3 mm, vias 0 -> 2
- net /Core/PC.CAR: track 1.00 -> 27.2 mm, vias 0 -> 1
- net BAT_SAMPLE_EN: track 0.00 -> 26.1 mm, vias 0 -> 2
- net /Core/PC.D0: track 1.00 -> 25.1 mm, vias 0 -> 1
- net /Core/PC.D3: track 0.00 -> 23.8 mm, vias 0 -> 2
- net /Core/PC.D2: track 3.91 -> 27.7 mm, vias 0 -> 2
- net /Core/PB.CB: track 3.91 -> 27.3 mm
- net /Core/PC.CA: track 0.00 -> 23.1 mm, vias 0 -> 1
- net /Core/PC.D1: track 0.00 -> 22.4 mm, vias 0 -> 1
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- added copper zone on F.Cu, net +3V3
- added copper zone on B.Cu, net GND_CORE

Commit message: Main PCB done
Parts:
- J21: moved to B.Cu
- moved J21 28.9 mm to (51.0, 0.00), turned to 90 degrees
- moved H5 1.00 mm to (27.2, -17.8)
- moved H6 1.00 mm to (27.2, 17.8)
- moved H7 1.00 mm to (62.8, 17.8)
- moved H8 1.00 mm to (62.8, -17.8)
- moved J10 1.00 mm to (45.0, 10.0)
- moved J11 1.00 mm to (61.3, 0.10)
- moved SW1 1.00 mm to (45.0, 0.00)
- moved SW2 1.00 mm to (31.5, 0.00)
- moved SW3 1.00 mm to (45.0, 13.5)
- moved SW4 1.00 mm to (58.5, 0.00)
- moved SW5 1.00 mm to (45.0, -13.5)
Connections:
- J20 pad 4: unconnected-(J20-Pin_4-Pad4) -> GND_CORE
- J20 pad 5: unconnected-(J20-Pin_5-Pad5) -> +3V3
- J20 pad 6: unconnected-(J20-Pin_6-Pad6) -> GND_CORE
- J21 pad 2: unconnected-(J21-Pin_2-Pad2) -> /Peripheral/USB_D-
- J21 pad 3: unconnected-(J21-Pin_3-Pad3) -> /Peripheral/USB_D+
- J21 pad 4: unconnected-(J21-Pin_4-Pad4) -> GND_PERI
- J21 pad 5: unconnected-(J21-Pin_5-Pad5) -> /Peripheral/+3V3
- J21 pad 6: unconnected-(J21-Pin_6-Pad6) -> GND_PERI
Routing:
- net /Core/VIN: track 182.5 -> 195.2 mm, vias 4 -> 5
- net (no net): track 46.9 -> 40.0 mm
- net +3V3: track 105.7 -> 111.0 mm, vias 9 -> 10
- net GND_CORE: track 126.2 -> 127.2 mm, vias 34 -> 113
Other:
- board size 86 x 40 mm -> 85 x 40 mm
- copper layers 4 -> 2

Commit message: PCB done
Parts:
- C27, C28, C29, R32, R33, R46, R47, U8: moved to B.Cu
- moved JP3 77.4 mm to (32.0, 13.5), turned to -90 degrees
- moved JP4 73.3 mm to (34.5, 13.5), turned to -90 degrees
- moved C35 70.6 mm to (29.8, 12.1), turned to -90 degrees
- moved JP5 69.3 mm to (37.0, 13.5), turned to -90 degrees
- moved R42 67.2 mm to (39.9, 14.6)
- moved R31 59.3 mm to (35.7, 2.90), turned to 180 degrees
- moved R39 56.3 mm to (39.9, 11.6), turned to 180 degrees
- moved R38 55.9 mm to (35.7, -0.10)
- moved R41 55.2 mm to (39.9, -12.0), turned to 180 degrees
- moved C27 55.0 mm to (42.8, 6.10), turned to 90 degrees
- moved U9 54.5 mm to (32.1, 8.36), turned to 90 degrees
- moved C32 53.8 mm to (39.9, 13.1)
- moved R46 53.3 mm to (42.0, 1.05)
- moved C31 52.8 mm to (35.7, 1.40), turned to 180 degrees
- moved D3 52.7 mm to (43.2, -4.25), turned to -90 degrees
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Connections:
- J10 pad 10: /Peripheral/LCD_MOSI -> /Peripheral/+3V3
- J10 pad 11: LCD_RST -> LCD_BL
- J10 pad 2: LCD_BL -> LCD_RST
- J10 pad 3: /Peripheral/+3V3 -> /Peripheral/LCD_MOSI
- J10 pad 4: /Peripheral/+3V3 -> /Peripheral/LCD_SCK
- J10 pad 5: GND_PERI -> /Peripheral/LCD_CS
- J10 pad 6: GND_PERI -> /Peripheral/LCD_DC
- J10 pad 7: /Peripheral/LCD_DC -> GND_PERI
- J10 pad 8: /Peripheral/LCD_CS -> GND_PERI
- J10 pad 9: /Peripheral/LCD_SCK -> /Peripheral/+3V3
- J21 pad 13: unconnected-(J21-Pin_13-Pad13) -> /Peripheral/I2C_SCL
- J21 pad 14: unconnected-(J21-Pin_14-Pad14) -> /Peripheral/I2C_SDA
- J21 pad 15: unconnected-(J21-Pin_15-Pad15) -> /Peripheral/PERI_INT
- J21 pad 16: unconnected-(J21-Pin_16-Pad16) -> /Peripheral/LCD_DC
- J21 pad 17: unconnected-(J21-Pin_17-Pad17) -> /Peripheral/LCD_MOSI
- J21 pad 18: unconnected-(J21-Pin_18-Pad18) -> /Peripheral/LCD_SCK
- J21 pad 19: unconnected-(J21-Pin_19-Pad19) -> /Peripheral/LCD_CS
- J21 pad 8: unconnected-(J21-Pin_8-Pad8) -> /Peripheral/BTN_CENTER
- U9 pad 10: BTN_LEFT -> BTN_BOTTOM
- U9 pad 11: BTN_BOTTOM -> BTN_RIGHT
- U9 pad 12: BTN_RIGHT -> BTN_LEFT
- U9 pad 14: unconnected-(U9-P1_4-Pad14) -> LCD_RST
- U9 pad 17: LCD_RST -> unconnected-(U9-P1_7-Pad17)
- U9 pad 5: IMU_INT1 -> unconnected-(U9-P0_0-Pad5)
- U9 pad 6: IMU_INT2 -> unconnected-(U9-P0_1-Pad6)
- U9 pad 7: unconnected-(U9-P0_2-Pad7) -> IMU_INT1
- U9 pad 8: unconnected-(U9-P0_3-Pad8) -> IMU_INT2
Routing:
- net /Peripheral/+3V3: track 0.00 -> 135.3 mm, vias 0 -> 8
- net GND_PERI: track 0.00 -> 75.2 mm, vias 0 -> 68
- net (no net): track 40.0 -> 0.00 mm, vias 12 -> 0
- net GND_CORE: track 127.2 -> 158.6 mm, vias 113 -> 123
- net /Peripheral/PERI_INT: track 0.00 -> 29.1 mm, vias 0 -> 1
- net /Peripheral/I2C_SCL: track 0.00 -> 27.7 mm, vias 0 -> 3
- net /Peripheral/I2C_SDA: track 0.00 -> 26.3 mm, vias 0 -> 3
- net BTN_RIGHT: track 0.00 -> 26.2 mm
- net BTN_TOP: track 0.00 -> 23.8 mm
- net IMU_INT2: track 0.00 -> 21.8 mm, vias 0 -> 1
- net LCD_BL: track 0.00 -> 20.0 mm, vias 0 -> 1
- net /Peripheral/BTN_CENTER_VBUS: track 0.00 -> 18.4 mm, vias 0 -> 1
- net LCD_RST: track 0.00 -> 17.8 mm, vias 0 -> 3
- net /Peripheral/VBUS: track 0.00 -> 15.4 mm, vias 0 -> 1
- net IMU_INT1: track 0.00 -> 15.0 mm, vias 0 -> 1
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- added copper zone on B.Cu, net GND_PERI
- added copper zone on F.Cu, net GND_PERI
Other:
- outline, holes or cut-outs redrawn
