File: hardware/SnapNodes_RP2/Core.kicad_sch (KiCad schematic)
At the start: 121 parts, among them J1 P_Female, J12 P_Female_Fallback, J13 P_Male_Fallback, J14 P_Female_Fallback, J15 P_Male_Fallback, J16 P_Female_Fallback, J17 P_Male_Fallback, J18 P_Female_Fallback, J19 P_Male_Fallback, J2 P_Male, J3 P_Female, J4 P_Male, J5 P_Female, J6 P_Male, J7 P_Female, J8 P_Male, J9 SWD, Q1 2N7002W, U1 RP2350_80QFN, U2 TPS62A01PDDC, U3 BQ24232RGT, U4 ESP-PSRAM64H, U6 PY25Q128HA-SSH, U7 74AHC1G04, Y1 12M

Commit message: PCB minor changes
Parts:
- C36: Link https://www.lcsc.com/product-detail/C45359895.html -> https://www.lcsc.com/product-detail/C20069326.html
- R19, R22, R23: Link https://www.lcsc.com/product-detail/C2906868.html -> https://www.lcsc.com/product-detail/C2906859.html
- R28, R29, R34: Link https://www.lcsc.com/product-detail/C2907002.html -> https://www.lcsc.com/product-detail/C2906980.html
Changed lines of the file:
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@@
 			)
 		)
-		(property "Link" "https://www.lcsc.com/product-detail/C2906868.html"
+		(property "Link" "https://www.lcsc.com/product-detail/C2906859.html"
 			(at 44.45 264.16 90)
 			(effects
@@
 			)
 		)
-		(property "Link" "https://www.lcsc.com/product-detail/C2906868.html"
+		(property "Link" "https://www.lcsc.com/product-detail/C2906859.html"
 			(at 149.86 134.62 90)
 			(effects
@@
 			)
 		)
-		(property "Link" "https://www.lcsc.com/product-detail/C2907002.html"
+		(property "Link" "https://www.lcsc.com/product-detail/C2906980.html"
 			(at 203.2 243.84 90)
 			(effects
@@
 			)
 		)
-		(property "Link" "https://www.lcsc.com/product-detail/C2906868.html"
+		(property "Link" "https://www.lcsc.com/product-detail/C2906859.html"
 			(at 118.11 226.06 90)
 			(effects
@@
 			)
 		)
-		(property "Link" "https://www.lcsc.com/product-detail/C2907002.html"
+		(property "Link" "https://www.lcsc.com/product-detail/C2906980.html"
 			(at 205.74 153.67 90)
 			(effects
@@
 			)
 		)
-		(property "Link" "https://www.lcsc.com/product-detail/C45359895.html"
+		(property "Link" "https://www.lcsc.com/product-detail/C20069326.html"
 			(at 251.46 241.3 0)
 			(effects
@@
 			)
 		)
-		(property "Link" "https://www.lcsc.com/product-detail/C2907002.html"
+		(property "Link" "https://www.lcsc.com/product-detail/C2906980.html"
 			(at 205.74 119.38 90)
 			(effects
